File: Synth_2.brd (EAGLE design)
At the start: 160 x 100 mm, 71 parts, among them IC1 DG409DJ, IC2 DG409DJ, IC3 DG409DJ, X1 POWER_SUPPLY

Commit message: Changes
Parts:
- added C6: (no value), rcl:C025-024X044
- added OSC_SUM_TRIM: (no value), pot:CT6
- added R41: (no value), rcl:0204/7
- PSOC_LOGIC: device con-phoenix-254:3POL254 -> con-phoenix-254:2POL254
- moved PSOC_LOGIC 0.57 mm to (86.7, 96.4), turned to 180 degrees
Connections:
- net +15V_PS: now also R41.2
- net +5V_PS: now also IC1.2, IC2.2, IC3.2, OSC_SUM_TRIM.A; no longer R8.1
- net COMPARATOR: now also C6.2, R41.1
- net GND_PS: now also C6.1
- net N$26: now also U$4.AMP_BIAS_1
- net N$54: now also OSC_SUM_TRIM.S, R8.1; no longer IC1.2, PSOC_LOGIC.1
- net N$6: now also PSOC_LOGIC.2; no longer PSOC_LOGIC.3
- net N$7: now also PSOC_LOGIC.1; no longer PSOC_LOGIC.2
- net SAWTOOTH: now also IC2.7; no longer IC2.6
- net TRIANGLE: now also IC2.6; no longer IC2.5

Commit message: Filter changes
Parts:
- added FILTER_RESONANCE: (no value), con-phoenix-254:2POL254
Connections:
- new net N$55: FILTER_RESONANCE.1, R20.2
- net N$21: now also FILTER_RESONANCE.2; no longer R20.2
Changed lines of the file:
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@@
 <attribute name="NAME" x="147.5994" y="78.232" size="0.9906" layer="25" ratio="10" rot="R270"/>
 <attribute name="POPULARITY" value="48" x="73.914" y="47.752" size="1.778" layer="27" rot="R270" display="off"/>
-<attribute name="SPICEPREFIX" value="10K" x="73.914" y="47.752" size="1.778" layer="27" rot="R270" display="off"/>
+<attribute name="SPICEPREFIX" value="5K" x="73.914" y="47.752" size="1.778" layer="27" rot="R270" display="off"/>
 <attribute name="VALUE" x="145.8214" y="77.3176" size="0.9906" layer="27" ratio="10" rot="R270"/>
 </element>
@@
 <attribute name="SPICEPREFIX" value="1.5nF" x="27.686" y="27.432" size="1.778" layer="27" rot="R90" display="off"/>
 <attribute name="VALUE" x="30.353" y="25.654" size="1.27" layer="27" ratio="10" rot="R90"/>
+</element>
+<element name="FILTER_RESONANCE" library="con-phoenix-254" library_urn="urn:adsk.eagle:library:172" package="2POL254" package3d_urn="urn:adsk.eagle:package:9320/1" value="" x="132.08" y="95.758" smashed="yes" rot="R180">
+<attribute name="MF" value="" x="132.08" y="95.758" size="1.778" layer="27" rot="R180" display="off"/>
+<attribute name="MPN" value="" x="132.08" y="95.758" size="1.778" layer="27" rot="R180" display="off"/>
+<attribute name="NAME" x="134.874" y="93.98" size="1.27" layer="25" rot="R180"/>
+<attribute name="OC_FARNELL" value="unknown" x="132.08" y="95.758" size="1.778" layer="27" rot="R180" display="off"/>
+<attribute name="OC_NEWARK" value="unknown" x="132.08" y="95.758" size="1.778" layer="27" rot="R180" display="off"/>
+<attribute name="POPULARITY" value="5" x="132.08" y="95.758" size="1.778" layer="27" rot="R180" display="off"/>
+<attribute name="VALUE" x="134.874" y="98.806" size="1.27" layer="27" rot="R180"/>
 </element>
 </elements>
@@
 <signal name="N$21">
 <contactref element="FILTER_TRIM" pad="E"/>
-<contactref element="R20" pad="2"/>
 <contactref element="R21" pad="2"/>
 <contactref element="U$4" pad="+IN_1"/>
-<wire x1="143.891" y1="71.882" x2="146.304" y2="71.882" width="0" layer="19" extent="1-1"/>
-<wire x1="153.162" y1="31.0896" x2="143.891" y2="71.882" width="0" layer="19" extent="1-1"/>
-<wire x1="127.889" y1="56.134" x2="153.162" y2="31.0896" width="0" layer="19" extent="1-1"/>
+<contactref element="FILTER_RESONANCE" pad="2"/>
+<wire x1="127.889" y1="56.134" x2="143.891" y2="71.882" width="0" layer="19" extent="1-1"/>
+<wire x1="153.162" y1="31.0896" x2="127.889" y2="56.134" width="0" layer="19" extent="1-1"/>
+<wire x1="130.81" y1="95.758" x2="127.889" y2="56.134" width="0" layer="19" extent="1-1"/>
 </signal>
 <signal name="N$22">
@@
 <wire x1="36.703" y1="8.509" x2="71.374" y2="73.533" width="0" layer="19" extent="1-1"/>
 </signal>
+<signal name="N$55">
+<contactref element="R20" pad="2"/>
+<contactref element="FILTER_RESONANCE" pad="1"/>
+<wire x1="133.35" y1="95.758" x2="146.304" y2="71.882" width="0" layer="19" extent="1-1"/>
+</signal>
 </signals>
