File: Synth_2.sch (EAGLE design)
At the start: 71 parts, among them IC1 DG409DJ, IC2 DG409DJ, IC3 DG409DJ, X1 POWER_SUPPLY

Commit message: Changes
Parts:
- added C6: (no value), rcl:C-EU025-024X044
- added OSC_SUM_TRIM: (no value), pot:TRIM_US-CT6
- added R41: (no value), rcl:R-US_0204/7
- PSOC_LOGIC: device con-phoenix-254:MPT3 -> con-phoenix-254:MPT2
- R16: SPICEPREFIX 20K -> 330K
- R17: SPICEPREFIX 10K -> 180K
- R26, R27, R28, R29, R7, R9: SPICEPREFIX 10K -> 100K
- R33: SPICEPREFIX 90K -> 10K
- R6: SPICEPREFIX 1K -> 1.5K
- R8: SPICEPREFIX 10K -> 90K
Connections:
- net +15V_PS: now also R41.2
- net +5V_PS: now also IC1.EN, IC2.EN, IC3.EN, OSC_SUM_TRIM.A; no longer R8.1
- net COMPARATOR: now also C6.2, R41.1
- net GND_PS: now also C6.1
- net N$26: now also U$4G$1.AMP_BIAS_1
- net N$54: now also OSC_SUM_TRIM.S, R8.1; no longer IC1.EN, PSOC_LOGIC-1.1
- net N$6: now also PSOC_LOGIC-2.1; no longer PSOC_LOGIC-3.1
- net N$7: now also PSOC_LOGIC-1.1; no longer PSOC_LOGIC-2.1
- net SAWTOOTH: now also IC2.S4A; no longer IC2.S3A
- net TRIANGLE: now also IC2.S3A; no longer IC2.S2A
Other:
- moved on the sheet: PSOC_LOGIC-1, PSOC_LOGIC-2, R16

Commit message: Filter changes
Parts:
- added FILTER_RESONANCE: (no value), con-phoenix-254:MPT2
- R20: SPICEPREFIX 10K -> 5K
Connections:
- new net N$55: FILTER_RESONANCE-1.1, R20.2
- net N$21: now also FILTER_RESONANCE-2.1; no longer R20.2
Changed lines of the file:
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@@
 <schematic_group name="VCA"/>
 <schematic_group name="OSCILLATOR"/>
+<schematic_group name="RESONANCE_CONTROL"/>
 </groups>
 <parts>
@@
 </pinmapping>
 </spice>
-<attribute name="SPICEPREFIX" value="10K"/>
+<attribute name="SPICEPREFIX" value="5K"/>
 </part>
 <part name="C4" library="rcl" library_urn="urn:adsk.eagle:library:334" deviceset="C-EU" device="025-024X044" package3d_urn="urn:adsk.eagle:package:23630/1">
@@
 <attribute name="SPICEPREFIX" value="1.5nF"/>
 </part>
+<part name="FILTER_RESONANCE" library="con-phoenix-254" library_urn="urn:adsk.eagle:library:172" deviceset="MPT2" device="" package3d_urn="urn:adsk.eagle:package:9320/1"/>
 </parts>
 <sheets>
@@
 <attribute name="VALUE" x="227.076" y="52.959" size="1.778" layer="96" rot="R180"/>
 <attribute name="SPICEPREFIX" x="231.14" y="53.34" size="1.778" layer="96" rot="R270"/>
+</instance>
+<instance part="FILTER_RESONANCE" gate="-1" x="365.76" y="-12.7" smashed="yes" rot="R270" grouprefs="RESONANCE_CONTROL">
+<attribute name="NAME" x="365.125" y="-16.256" size="1.778" layer="95" rot="R270"/>
+</instance>
+<instance part="FILTER_RESONANCE" gate="-2" x="363.22" y="-12.7" smashed="yes" rot="R270" grouprefs="RESONANCE_CONTROL">
+<attribute name="NAME" x="362.585" y="-16.256" size="1.778" layer="95" rot="R270"/>
+<attribute name="VALUE" x="359.918" y="-11.684" size="1.778" layer="96" rot="R270"/>
 </instance>
 </instances>
@@
 <wire x1="358.14" y1="48.26" x2="365.76" y2="48.26" width="0.1524" layer="91" grouprefs="FILTER"/>
 <wire x1="365.76" y1="48.26" x2="365.76" y2="60.96" width="0.1524" layer="91" grouprefs="FILTER"/>
-<pinref part="R20" gate="G$1" pin="2"/>
 <wire x1="358.14" y1="48.26" x2="358.14" y2="43.18" width="0.1524" layer="91" grouprefs="FILTER"/>
-<wire x1="358.14" y1="43.18" x2="368.3" y2="43.18" width="0.1524" layer="91" grouprefs="FILTER"/>
+<wire x1="358.14" y1="43.18" x2="363.22" y2="43.18" width="0.1524" layer="91" grouprefs="FILTER"/>
 <junction x="358.14" y="48.26" grouprefs="FILTER"/>
 <pinref part="R21" gate="G$1" pin="2"/>
@@
 <junction x="358.14" y="43.18" grouprefs="FILTER"/>
 <pinref part="U$4" gate="G$1" pin="+IN_1"/>
+<pinref part="FILTER_RESONANCE" gate="-2" pin="1"/>
+<wire x1="363.22" y1="-10.16" x2="363.22" y2="43.18" width="0.1524" layer="91"/>
 </segment>
 </net>
@@
 </segment>
 </net>
+<net name="N$55" class="0">
+<segment>
+<pinref part="R20" gate="G$1" pin="2"/>
+<wire x1="365.76" y1="43.18" x2="368.3" y2="43.18" width="0.1524" layer="91" grouprefs="FILTER"/>
+<pinref part="FILTER_RESONANCE" gate="-1" pin="1"/>
+<wire x1="365.76" y1="-10.16" x2="365.76" y2="43.18" width="0.1524" layer="91"/>
+</segment>
+</net>
